File: Sequencer/KiCAD/sequencer.kicad_sch (KiCad schematic)
At the start: 22 parts, among them J1 12V -13,8V DC, J2 MCU 11, J3 GX12, Q1 BC237, Q2 BC237, Q3 PNP

Commit message: 3.7.26
Parts:
- removed J2: MCU 11, Connector_PinHeader_2.54mm:PinHeader_1x01_P2.54mm_Horizontal, symbol Connector:Screw_Terminal_01x01
- added J2: MCU, Connector_PinHeader_2.54mm:PinHeader_1x02_P2.54mm_Horizontal, symbol Connector:Screw_Terminal_01x02
- added J4: LNA, Connector_PinHeader_2.54mm:PinHeader_1x02_P2.54mm_Horizontal, symbol Connector:Screw_Terminal_01x02
- J1: value 12V -13,8V DC -> 12V
- Q1, Q2: footprint Package_TO_SOT_THT:TO-92_Inline -> Package_TO_SOT_THT:TO-92L_HandSolder
Connections:
- net GND: now also J2.2 (Pin_2), J4.1 (Pin_1)
- net at R1.2: now also J2.1 (Pin_1)
- net +VIN renamed +12V
- net +12V: no longer Q3.3 (E), R7.1
- new net +LNA: J4.2 (Pin_2), Q3.3 (E), R7.1
Other:
- moved on the sheet: D1, J1, Q2, R2, R4, R5, R6, R7, R8
